Commit message: Fixed some inertias in talos model and using this urdf for cartesio

File: robots/talos.urdf (robot description, URDF)
Before this commit: robot talos, 55 links, 54 joints
Links:
- link imu_link: mass 0.01 -> None; geometry 
- link left_sole_link: mass 0.01 -> None
- link leg_left_6_link: geometry collision box size=0.21 0.13 0.02; visual mesh filename=package://talos_description/meshes/v2/ankle_X_lo_res.stl scale=1 1 1
- link leg_right_6_link: geometry collision box size=0.21 0.13 0.02; visual mesh filename=package://talos_description/meshes/v2/ankle_X_lo_res.stl scale=1 -1 1
- link rgbd_link: mass 0.01 -> None; geometry 
- link rgbd_optical_frame: mass 0.01 -> None
- link right_sole_link: mass 0.01 -> None
- link wrist_left_ft_tool_link: mass 0.001 -> None; geometry 
- link wrist_right_ft_link: mass 0.095 -> None; geometry 
- link wrist_right_ft_tool_link: mass 0.001 -> None; geometry 
Joints:
- joint reference: origin xyz=0 0 1 -> xyz=0 0 0.1

File: robots/talos.urdf.xacro (robot description, xacro)
@@ -1,5 +1,6 @@
 <?xml version='1.0' encoding='utf-8'?>
 <robot xmlns:xacro="http://www.ros.org/wiki/xacro" name="talos">
-<xacro:include filename="$(find talos_description)/robots/talos_full_fake_grippers.urdf.xacro"/>
+<!--xacro:include filename="$(find talos_description)/robots/talos_full_fake_grippers.urdf.xacro"/-->
+<xacro:include filename="$(find talos_cartesio_config)/robots/talos.urdf"/>
 <link name="world"/>
   <joint name="reference" type="floating">
